File: Macro-Board.kicad_sch (KiCad schematic)
At the start: 62 parts, among them J1 esp32row1, J2 esp32row1, K1 KEYSW, K10 KEYSW, K11 KEYSW, K12 KEYSW, K13 KEYSW, K14 KEYSW, K15 KEYSW, K16 KEYSW, K17 KEYSW, K18 KEYSW, K19 KEYSW, K2 KEYSW, K20 KEYSW, K21 KEYSW, K22 KEYSW, K23 KEYSW, K24 KEYSW, K25 KEYSW, K27 KEYSW, K28 KEYSW, K29 KEYSW, K3 KEYSW, K30 KEYSW, K4 KEYSW, K5 KEYSW, K6 KEYSW, K7 KEYSW, K8 KEYSW, K9 KEYSW, SW26 RotaryEncoder_Alps_EC11E-Swit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

Commit message: Idfk
Connections:
- net GPIO18 is gone; now on net EncoderA: J2.11 (Pin_11)
- net EncoderA: no longer J2.9 (Pin_9)
- net EncoderB: now also J2.12 (Pin_12); no longer J2.10 (Pin_10)
- net GND1: now also SW26.C
- net GND4: no longer SW26.C
- net GPIO01: now also K1.1, K11.1, K16.1, K21.1, K6.1, SW26.S1
- net GPIO02: now also K12.1, K17.1, K2.1, K22.1, K27.1, K7.1
- net GPIO04: no longer D26.1 (K), D27.1 (K), D28.1 (K), D29.1 (K), D30.1 (K)
- net GPIO05: now also D21.1 (K), D22.1 (K), D23.1 (K), D24.1 (K), D25.1 (K); no longer K10.1, K15.1, K20.1, K25.1, K30.1, K5.1
- net GPIO06: now also D16.1 (K), D17.1 (K), D18.1 (K), D19.1 (K), D20.1 (K); no longer K14.1, K19.1, K24.1, K29.1, K4.1, K9.1
- net GPIO07: now also D11.1 (K), D12.1 (K), D13.1 (K), D14.1 (K), D15.1 (K); no longer K13.1, K18.1, K23.1, K28.1, K3.1, K8.1
- net GPIO15: now also D10.1 (K), D6.1 (K), D7.1 (K), D8.1 (K), D9.1 (K); no longer K12.1, K17.1, K2.1, K22.1, K27.1, K7.1
- net GPIO38: no longer D21.1 (K), D22.1 (K), D23.1 (K), D24.1 (K), D25.1 (K)
- net GPIO39: no longer D16.1 (K), D17.1 (K), D18.1 (K), D19.1 (K), D20.1 (K)
- net GPIO40: now also K10.1, K15.1, K20.1, K25.1, K30.1, K5.1; no longer D11.1 (K), D12.1 (K), D13.1 (K), D14.1 (K), D15.1 (K)
- net GPIO41: now also K14.1, K19.1, K24.1, K29.1, K4.1, K9.1; no longer D10.1 (K), D6.1 (K), D7.1 (K), D8.1 (K), D9.1 (K)
- net GPIO42: now also K13.1, K18.1, K23.1, K28.1, K3.1, K8.1; no longer D1.1 (K), D2.1 (K), D3.1 (K), D4.1 (K), D5.1 (K)
- removed net GPIO08: J2.12 (Pin_12), K1.1, K11.1, K16.1, K21.1, K6.1, SW26.S1
- new net GPIO16: D1.1 (K), D2.1 (K), D3.1 (K), D4.1 (K), D5.1 (K), J2.9 (Pin_9)
- new net GPIO17: D26.1 (K), D27.1 (K), D28.1 (K), D29.1 (K), D30.1 (K), J2.10 (Pin_10)
Other:
- moved on the sheet: J1, J2
