File: Macro-Board.kicad_sch (KiCad schematic)
At the start: 62 parts, among them J1 esp32row1, J2 esp32row1, K1 KEYSW, K10 KEYSW, K11 KEYSW, K12 KEYSW, K13 KEYSW, K14 KEYSW, K15 KEYSW, K16 KEYSW, K17 KEYSW, K18 KEYSW, K19 KEYSW, K2 KEYSW, K20 KEYSW, K21 KEYSW, K22 KEYSW, K23 KEYSW, K24 KEYSW, K25 KEYSW, K27 KEYSW, K28 KEYSW, K29 KEYSW, K3 KEYSW, K30 KEYSW, K4 KEYSW, K5 KEYSW, K6 KEYSW, K7 KEYSW, K8 KEYSW, K9 KEYSW, SW26 RotaryEncoder_Alps_EC11E-Swit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

Commit message: PC modifications ffs
Connections:
- net EncoderA: now also J2.10 (Pin_10); no longer J2.9 (Pin_9)
- net EncoderB: now also J2.9 (Pin_9); no longer J2.10 (Pin_10)
- net GND1: now also SW26.C
- net GND4: no longer SW26.C
- net GPIO04: now also D21.1 (K), D22.1 (K), D23.1 (K), D24.1 (K), D25.1 (K); no longer D26.1 (K), D27.1 (K), D28.1 (K), D29.1 (K), D30.1 (K)
- net GPIO05: now also D16.1 (K), D17.1 (K), D18.1 (K), D19.1 (K), D20.1 (K); no longer K10.1, K15.1, K20.1, K25.1, K30.1, K5.1
- net GPIO06: now also D11.1 (K), D12.1 (K), D13.1 (K), D14.1 (K), D15.1 (K); no longer K14.1, K19.1, K24.1, K29.1, K4.1, K9.1
- net GPIO07: now also D10.1 (K), D6.1 (K), D7.1 (K), D8.1 (K), D9.1 (K); no longer K13.1, K18.1, K23.1, K28.1, K3.1, K8.1
- net GPIO08: now also D26.1 (K), D27.1 (K), D28.1 (K), D29.1 (K), D30.1 (K); no longer K1.1, K11.1, K16.1, K21.1, K6.1, SW26.S1
- net GPIO15: now also D1.1 (K), D2.1 (K), D3.1 (K), D4.1 (K), D5.1 (K); no longer K12.1, K17.1, K2.1, K22.1, K27.1, K7.1
- net GPIO38: now also K10.1, K15.1, K20.1, K25.1, K30.1, K5.1; no longer D21.1 (K), D22.1 (K), D23.1 (K), D24.1 (K), D25.1 (K)
- net GPIO39: now also K14.1, K19.1, K24.1, K29.1, K4.1, K9.1; no longer D16.1 (K), D17.1 (K), D18.1 (K), D19.1 (K), D20.1 (K)
- net GPIO40: now also K13.1, K18.1, K23.1, K28.1, K3.1, K8.1; no longer D11.1 (K), D12.1 (K), D13.1 (K), D14.1 (K), D15.1 (K)
- net GPIO41: now also K12.1, K17.1, K2.1, K22.1, K27.1, K7.1; no longer D10.1 (K), D6.1 (K), D7.1 (K), D8.1 (K), D9.1 (K)
- net GPIO42: now also K1.1, K11.1, K16.1, K21.1, K6.1, SW26.S1; no longer D1.1 (K), D2.1 (K), D3.1 (K), D4.1 (K), D5.1 (K)
Changed lines of the file:
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@@
+		)
+	)
+	(label "col4"
+		(at 438.15 279.4 0)
+		(effects
+			(font
+				(size 1.27 1.27)
+			)
+			(justify left bottom)
+		)
+	)
+	(label "row4"
+		(at 438.15 228.6 0)
+		(effects
+			(font
+				(size 1.27 1.27)
+			)
+			(justify left bottom)
 		)
 	)
@@
 		)
 	)
-	(label "row0"
-		(at 438.15 226.06 0)
-		(effects
-			(font
-				(size 1.27 1.27)
-			)
-			(justify left bottom)
-		)
-	)
 	(label "GPIO02"
 		(at 434.34 220.98 180)
@@
 		)
 	)
-	(label "row1"
-		(at 438.15 289.56 0)
+	(label "GND1"
+		(at 533.4 273.05 0)
 		(effects
 			(font
@@
 		)
 	)
-	(label "col1"
-		(at 438.15 254 0)
-		(effects
-			(font
-				(size 1.27 1.27)
-			)
-			(justify left bottom)
-		)
-	)
 	(label "GPIO18"
 		(at 434.34 261.62 180)
@@
 		)
 	)
-	(label "col4"
-		(at 438.15 228.6 0)
-		(effects
-			(font
-				(size 1.27 1.27)
-			)
-			(justify left bottom)
-		)
-	)
 	(label "GPIO14"
 		(at 393.7 264.16 0)
@@
 		)
 	)
+	(label "row2"
+		(at 438.15 233.68 0)
+		(effects
+			(font
+				(size 1.27 1.27)
+			)
+			(justify left bottom)
+		)
+	)
 	(label "GPIO09"
 		(at 393.7 251.46 0)
@@
 		)
 	)
+	(label "col1"
+		(at 438.15 287.02 0)
+		(effects
+			(font
+				(size 1.27 1.27)
+			)
+			(justify left bottom)
+		)
+	)
 	(label "GPIO15"
 		(at 455.93 198.12 180)
@@
 		)
 	)
-	(label "EncoderA"
-		(at 434.34 256.54 0)
-		(effects
-			(font
-				(size 1.27 1.27)
-			)
-			(justify left bottom)
-		)
-	)
 	(label "3.3v1"
 		(at 393.7 215.9 0)
@@
 		)
 	)
+	(label "col2"
+		(at 438.15 284.48 0)
+		(effects
+			(font
+				(size 1.27 1.27)
+			)
+			(justify left bottom)
+		)
+	)
 	(label "GPIO20"
 		(at 455.93 218.44 180)
@@
 		)
 	)
+	(label "row3"
+		(at 438.15 231.14 0)
+		(effects
+			(font
+				(size 1.27 1.27)
+			)
+			(justify left bottom)
+		)
+	)
+	(label "EncoderB"
+		(at 434.34 256.54 0)
+		(effects
+			(font
+				(size 1.27 1.27)
+			)
+			(justify left bottom)
+		)
+	)
 	(label "GPIO37"
 		(at 434.34 276.86 180)
@@
 		)
 	)
-	(label "GND4"
-		(at 533.4 273.05 180)
-		(effects
-			(font
-				(size 1.27 1.27)
-			)
-			(justify right bottom)
-		)
-	)
-	(label "row3"
-		(at 438.15 284.48 0)
-		(effects
-			(font
-				(size 1.27 1.27)
-			)
-			(justify left bottom)
-		)
-	)
 	(label "GPIO48"
 		(at 410.21 254 180)
@@
 		)
 	)
-	(label "col3"
-		(at 438.15 231.14 0)
-		(effects
-			(font
-				(size 1.27 1.27)
-			)
-			(justify left bottom)
-		)
-	)
 	(label "GPIO07"
 		(at 434.34 233.68 180)
@@
 		)
 	)
-	(label "row4"
-		(at 438.15 281.94 0)
-		(effects
-			(font
-				(size 1.27 1.27)
-			)
-			(justify left bottom)
-		)
-	)
 	(label "col0"
 		(at 543.56 289.56 0)
@@
 		)
 	)
-	(label "row2"
-		(at 438.15 287.02 0)
+	(label "col3"
+		(at 438.15 281.94 0)
 		(effects
 			(font
@@
 		)
 	)
-	(label "row5"
-		(at 438.15 279.4 0)
-		(effects
-			(font
-				(size 1.27 1.27)
-			)
-			(justify left bottom)
-		)
-	)
 	(label "GPIO21"
 		(at 410.21 259.08 180)
@@
 		)
 	)
+	(label "EncoderA"
+		(at 434.34 259.08 0)
+		(effects
+			(font
+				(size 1.27 1.27)
+			)
+			(justify left bottom)
+		)
+	)
 	(label "GPIO11"
 		(at 455.93 203.2 180)
@@
 		)
 	)
+	(label "col0"
+		(at 438.15 289.56 0)
+		(effects
+			(font
+				(size 1.27 1.27)
+			)
+			(justify left bottom)
+		)
+	)
 	(label "GPIO40"
 		(at 434.34 284.48 180)
@@
 		)
 	)
+	(label "row1"
+		(at 438.15 254 0)
+		(effects
+			(font
+				(size 1.27 1.27)
+			)
+			(justify left bottom)
+		)
+	)
 	(label "GPIO43"
 		(at 410.21 218.44 180)
@@
 		)
 	)
-	(label "col0"
-		(at 438.15 236.22 0)
-		(effects
-			(font
-				(size 1.27 1.27)
-			)
-			(justify left bottom)
-		)
-	)
 	(label "GPIO21"
 		(at 434.34 269.24 180)
@@
 		)
 	)
-	(label "col2"
-		(at 438.15 233.68 0)
-		(effects
-			(font
-				(size 1.27 1.27)
-			)
-			(justify left bottom)
-		)
-	)
 	(label "GPIO36"
 		(at 434.34 274.32 180)
@@
 		)
 	)
+	(label "row0"
+		(at 438.15 236.22 0)
+		(effects
+			(font
+				(size 1.27 1.27)
+			)
+			(justify left bottom)
+		)
+	)
 	(label "RST"
 		(at 393.7 220.98 0)
@@
 		)
 	)
-	(label "EncoderB"
-		(at 434.34 259.08 0)
-		(effects
-			(font
-				(size 1.27 1.27)
-			)
-			(justify left bottom)
-		)
-	)
 	(label "GPIO12"
 		(at 434.34 246.38 180)
@@
 		)
 	)
+	(label "row5"
+		(at 438.15 226.06 0)
+		(effects
+			(font
+				(size 1.27 1.27)
+			)
+			(justify left bottom)
+		)
+	)

Commit message: 3x3 mod
Parts:
- removed D10, D11, D12, D13, D14, D15, D16, D17, D18, D19, D20, D21, D22, D23, D24, D25, D29, D30, D4, D5, D9: 1N4148W, Diode_SMD:D_SOD-123, symbol Diode:1N4148W
- removed K10, K11, K12, K13, K14, K15, K16, K17, K18, K19, K20, K21, K22, K23, K24, K25, K29, K30, K4, K5, K9: KEYSW, PCM_Switch_Keyboard_Hotswap_Kailh:SW_Hotswap_Kailh_MX_Plated_1.00u, symbol keyboard_parts:KEYSW
Connections:
- net EncoderA: now also J2.12 (Pin_12); no longer J2.10 (Pin_10)
- net EncoderB: now also J2.10 (Pin_10); no longer J2.9 (Pin_9)
- net GPIO08 renamed GPIO16
- net GPIO16: now also J2.9 (Pin_9); no longer J2.12 (Pin_12)
