File: Macro-Board.kicad_pcb (KiCad board)
At the start: 2 copper layers, 152.4 x 133.3 mm, 62 parts, among them J1 esp32row1, J2 esp32row1, K1 KEYSW, K10 KEYSW, K11 KEYSW, K12 KEYSW, K13 KEYSW, K14 KEYSW, K15 KEYSW, K16 KEYSW, K17 KEYSW, K18 KEYSW, K19 KEYSW, K2 KEYSW, K20 KEYSW, K21 KEYSW, K22 KEYSW, K23 KEYSW, K24 KEYSW, K25 KEYSW, K27 KEYSW, K28 KEYSW, K29 KEYSW, K3 KEYSW, K30 KEYSW, K4 KEYSW, K5 KEYSW, K6 KEYSW, K7 KEYSW, K8 KEYSW, K9 KEYSW, SW26 RotaryEncoder_Alps_EC11E-Swit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

Commit message: PC modifications ffs
Parts:
- moved J1 3.90 mm to (-39.4, -31.6)
- moved J2 3.90 mm to (-14.0, 21.8)
Connections:
- D1 pad 1: /GPIO42 -> /GPIO15
- D10 pad 1: /GPIO41 -> /GPIO07
- D11 pad 1: /GPIO40 -> /GPIO06
- D12 pad 1: /GPIO40 -> /GPIO06
- D13 pad 1: /GPIO40 -> /GPIO06
- D14 pad 1: /GPIO40 -> /GPIO06
- D15 pad 1: /GPIO40 -> /GPIO06
- D16 pad 1: /GPIO39 -> /GPIO05
- D17 pad 1: /GPIO39 -> /GPIO05
- D18 pad 1: /GPIO39 -> /GPIO05
- D19 pad 1: /GPIO39 -> /GPIO05
- D2 pad 1: /GPIO42 -> /GPIO15
- D20 pad 1: /GPIO39 -> /GPIO05
- D21 pad 1: /GPIO38 -> /GPIO04
- D22 pad 1: /GPIO38 -> /GPIO04
- D23 pad 1: /GPIO38 -> /GPIO04
- D24 pad 1: /GPIO38 -> /GPIO04
- D25 pad 1: /GPIO38 -> /GPIO04
- D26 pad 1: /GPIO04 -> /GPIO08
- D27 pad 1: /GPIO04 -> /GPIO08
- D28 pad 1: /GPIO04 -> /GPIO08
- D29 pad 1: /GPIO04 -> /GPIO08
- D3 pad 1: /GPIO42 -> /GPIO15
- D30 pad 1: /GPIO04 -> /GPIO08
- D4 pad 1: /GPIO42 -> /GPIO15
- D5 pad 1: /GPIO42 -> /GPIO15
- D6 pad 1: /GPIO41 -> /GPIO07
- D7 pad 1: /GPIO41 -> /GPIO07
- D8 pad 1: /GPIO41 -> /GPIO07
- D9 pad 1: /GPIO41 -> /GPIO07
- J2 pad 10: /EncoderB -> /EncoderA
- J2 pad 9: /EncoderA -> /EncoderB
- K1 pad 1: /GPIO08 -> /GPIO42
- K10 pad 1: /GPIO05 -> /GPIO38
- K11 pad 1: /GPIO08 -> /GPIO42
- K12 pad 1: /GPIO15 -> /GPIO41
- K13 pad 1: /GPIO07 -> /GPIO40
- K14 pad 1: /GPIO06 -> /GPIO39
- K15 pad 1: /GPIO05 -> /GPIO38
- K16 pad 1: /GPIO08 -> /GPIO42
- K17 pad 1: /GPIO15 -> /GPIO41
- K18 pad 1: /GPIO07 -> /GPIO40
- K19 pad 1: /GPIO06 -> /GPIO39
- K2 pad 1: /GPIO15 -> /GPIO41
- K20 pad 1: /GPIO05 -> /GPIO38
- K21 pad 1: /GPIO08 -> /GPIO42
- K22 pad 1: /GPIO15 -> /GPIO41
- K23 pad 1: /GPIO07 -> /GPIO40
- K24 pad 1: /GPIO06 -> /GPIO39
- K25 pad 1: /GPIO05 -> /GPIO38
- K27 pad 1: /GPIO15 -> /GPIO41
- K28 pad 1: /GPIO07 -> /GPIO40
- K29 pad 1: /GPIO06 -> /GPIO39
- K3 pad 1: /GPIO07 -> /GPIO40
- K30 pad 1: /GPIO05 -> /GPIO38
- K4 pad 1: /GPIO06 -> /GPIO39
- K5 pad 1: /GPIO05 -> /GPIO38
- K6 pad 1: /GPIO08 -> /GPIO42
- K7 pad 1: /GPIO15 -> /GPIO41
- K8 pad 1: /GPIO07 -> /GPIO40
- K9 pad 1: /GPIO06 -> /GPIO39
- SW26 pad C: /GND4 -> /GND1
- SW26 pad S1: /GPIO08 -> /GPIO42
Routing:
- net /GPIO05: track 297.7 -> 130.4 mm, vias 6 -> 0
- net /GPIO06: track 277.8 -> 114.5 mm, vias 6 -> 0
- net /GPIO07: track 258.0 -> 97.4 mm, vias 6 -> 0
- net /GPIO38: track 180.8 -> 328.6 mm, vias 0 -> 6
- net /GPIO39: track 161.4 -> 305.5 mm, vias 0 -> 6
- net /GPIO40: track 142.7 -> 282.6 mm, vias 0 -> 6
- net /GPIO41: track 123.1 -> 259.8 mm, vias 0 -> 6
- net /GPIO15: track 238.2 -> 105.0 mm, vias 6 -> 0
- net /GPIO42: track 103.9 -> 236.7 mm, vias 0 -> 6
- net /GPIO08: track 218.3 -> 128.5 mm, vias 6 -> 0
- net /GPIO04: track 93.3 -> 146.7 mm
- net /EncoderA: track 5.19 -> 25.1 mm
- net /GND1: track 0.00 -> 19.8 mm
- net /GND4: track 19.0 -> 0.00 mm
- net /EncoderB: track 10.0 -> 23.5 mm
Other:
- board size 152.4 x 133.3 mm -> 147.1 x 133.3 mm

Commit message: 3x3 mod
Parts:
- removed D10, D11, D12, D13, D14, D15, D16, D17, D18, D19, D20, D21, D22, D23, D24, D25, D29, D30, D4, D5, D9: 1N4148W, Diode_SMD:D_SOD-123
- removed K10, K11, K12, K13, K14, K15, K16, K17, K18, K19, K20, K21, K22, K23, K24, K25, K29, K30, K4, K5, K9: KEYSW, PCM_Switch_Keyboard_Hotswap_Kailh:SW_Hotswap_Kailh_MX_Plated_1.00u
- moved D6 5.45 mm to (-3.62, 9.78)
- moved D7 5.45 mm to (15.4, 9.78)
- moved K6 5.45 mm to (1.38, 13.8)
- moved K7 5.45 mm to (20.4, 13.8)
- moved D8 5.45 mm to (34.5, 9.78)
- moved K8 5.45 mm to (39.5, 13.8)
- moved D1 5.45 mm to (-3.62, -9.27)
- moved D2 5.45 mm to (15.4, -9.27)
- moved D26 5.45 mm to (5.93, -28.5)
- moved D27 5.45 mm to (15.4, -28.3)
- moved K1 5.45 mm to (1.38, -5.27)
- moved K2 5.45 mm to (20.4, -5.27)
- moved K27 5.45 mm to (20.4, -24.3)
- moved SW26 5.45 mm to (1.38, -24.3)
- moved D28 5.45 mm to (34.5, -28.3)
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Connections:
- D26 pad 1: /GPIO08 -> /GPIO16
- D27 pad 1: /GPIO08 -> /GPIO16
- D28 pad 1: /GPIO08 -> /GPIO16
- J2 pad 10: /EncoderA -> /EncoderB
- J2 pad 12: /GPIO08 -> /EncoderA
- J2 pad 9: /EncoderB -> /GPIO16
Routing:
- net /GPIO38: track 328.6 -> 0.00 mm, vias 6 -> 0
- net /GPIO39: track 305.5 -> 0.00 mm, vias 6 -> 0
- net /GPIO04: track 146.7 -> 0.00 mm
- net /GPIO05: track 130.4 -> 0.00 mm
- net /GPIO08: track 128.5 -> 0.00 mm
- net /GPIO40: track 282.6 -> 160.8 mm, vias 6 -> 3
- net /GPIO41: track 259.8 -> 138.1 mm, vias 6 -> 3
- net /GPIO42: track 236.7 -> 117.5 mm, vias 6 -> 3
- net /GPIO06: track 114.5 -> 0.00 mm
- net /GPIO16: track 0.00 -> 78.7 mm
- net /GPIO07: track 97.4 -> 53.9 mm
- net /GPIO15: track 105.0 -> 66.1 mm
- net Net-(D23-A): track 9.75 -> 0.00 mm
- net Net-(D13-A): track 9.75 -> 0.00 mm
- net Net-(D22-A): track 9.75 -> 0.00 mm
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Other:
- board size 147.1 x 133.3 mm -> 110.6 x 68.5 mm
